File: Flight-Computer/Flight-Computer.kicad_sch (KiCad schematic)
At the start: 40 parts, among them J1 Jumper_NO, J2 Jumper_NO, P1 647676-2, P2 1546551-2, P3 3220-20-0200-00, U1 STM32H750VBTx, U2 LMS8117AMP-3.3_NOPB, Y1 ECS-240-18-33-JGN-TR

Commit message: test
Other:
- added sheet Revision 3 Modifications (Rev3.kicad_sch)
Changed lines of the file:
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@@
 	(label "PIN_HARN"
 		(at 200.66 66.675 0)
+		(fields_autoplaced yes)
 		(effects
 			(font
@@
 	(label "PIN_SCREW"
 		(at 200.025 81.28 0)
+		(fields_autoplaced yes)
 		(effects
 			(font
@@
 				)
 			)
+		)
+	)
+	(sheet
+		(at 205.74 168.91)
+		(size 25.4 10.16)
+		(stroke
+			(width 0.1524)
+			(type solid)
+		)
+		(fill
+			(color 0 0 0 0.0000)
+		)
+		(property "Sheetname" "Revision 3 Modifications"
+			(at 205.994 170.688 0)
+			(effects
+				(font
+					(size 1.27 1.27)
+				)
+				(justify left bottom)
+			)
+		)
+		(property "Sheetfile" "Rev3.kicad_sch"
+			(at 205.74 177.292 0)
+			(effects
+				(font
+					(size 1.27 1.27)
+				)
+				(justify left top)
+			)
+		)
+		(instances
+			(project "Flight-Computer"
+				(path "/15d2e012-e166-422c-a8f3-0484b565dd65"
+					(page "4")
+				)
+			)
