File: Flight-Computer/Rev3.kicad_sch (KiCad schematic)
At the start: 2 parts, among them P11 440054-3, U14 MX25V5126FM1I

Commit message: test
Changed lines of the file:
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@@
 		(on_board yes)
 		(dnp no)
+		(fields_autoplaced yes)
 		(property "Reference" "U14"
 			(at 45.466 19.304 0)
@@
 		)
 		(property "Value" "MX25V5126FM1I"
-			(at 45.212 21.59 0)
+			(at 45.974 21.844 0)
 			(effects
 				(font
